File: hardware/uCKicad/uCKicad.kicad_pcb (KiCad board)
At the start: 2 copper layers, 62 x 52 mm, 27 parts, among them J1 Conn_02x07_Odd_Even, J2 INPUT, J3 OUTPUT, J4 POWER, U1 BU33SD5WG-TR, U2 MCP4801, U3 STM32L021K4Tx

Commit message: Routage
Parts:
- moved C8 3.93 mm to (117.4, 119.4), turned to 180 degrees
- moved L1 3.56 mm to (100.0, 102.1), turned to -90 degrees
- moved C9 3.54 mm to (117.3, 123.2), turned to 180 degrees
- moved J1 1.80 mm to (128.5, 94.0)
- moved C5 1.70 mm to (108.0, 104.4)
- moved C7 1.70 mm to (104.0, 104.3)
- moved U2 1.07 mm to (116.3, 114.0), turned to 180 degrees
Connections:
- net Net-(R3-Pad1) renamed /BOOT0
- C11 pad 2: Net-(C11-Pad2) -> GND
- C6 pad 2: Net-(C11-Pad2) -> GND
- U1 pad 2: Net-(C11-Pad2) -> GND
Routing:
- net +3.3V: track 0.00 -> 78.9 mm
- net +3.3VA: track 0.00 -> 40.9 mm
- net DAC_OUT: track 0.00 -> 38.6 mm, vias 0 -> 2
- net USART2_RX: track 0.00 -> 29.1 mm, vias 0 -> 2
- net ADC_IN1: track 0.00 -> 28.4 mm, vias 0 -> 2
- net USART2_TX: track 0.00 -> 24.3 mm, vias 0 -> 2
- net NRST: track 0.00 -> 23.5 mm, vias 0 -> 2
- net +5V: track 0.00 -> 13.5 mm
- net DAC_nCS: track 0.00 -> 8.89 mm
- net SWCLK: track 0.00 -> 8.74 mm
- net SWDIO: track 0.00 -> 8.49 mm
- net SPI1_SCK: track 0.00 -> 7.20 mm
- net Net-(D1-Pad1): track 0.00 -> 6.56 mm
- net LED_STATUS: track 0.00 -> 5.38 mm
- net /BOOT0: track 0.00 -> 5.24 mm
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- added copper zone on B.Cu, net GND
- added copper zone on F.Cu, net GND
Other:
- rule pad_to_mask_clearance: 0 -> 0.1
- board text added: "THOMAS Farima NOYON Yaëlle"
